File: CARL-Air-Brake-Peripheral-Devices-Hardware.kicad_sch (KiCad schematic)
At the start: 47 parts, among them J1 ICSP, J2 USB, J3 Raspberry Pi, J4 Servo power, J5 Servo port, P1 BMP388, P2 BMP388, P3 BNO055, P4 BNO055, Q1 BSS138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

Commit message: Assigned footprints
Assigned footprints to all components in circuit schematic.
Parts:
- C1, C2, C3, C4, C5, C6, C7, C8: footprint (none) -> Local_Capacitor_SMD:Cap_Ceramic_0603
- D1, D2, D3: footprint (none) -> Local_Diode_SMD:Diode_DO-214AB_SMC
- D4, D5, D6, D7, D8, D9: footprint (none) -> Local_LED_SMD:LED_0603
- J1: footprint (none) -> Local_Connector_PinHeader:PinHead_02x03_Pitch2.54mm_Bot3.00mm_Top6.00mm_Shroud2.50mm
- J2: footprint (none) -> Local_Connector_USB:USB_Micro_B_Recp_Wuerth_629105136821
- J3: footprint (none) -> Local_Connector_SocketHeader:SockHead_02x20_Pitch2.54mm_Bot3.10mm_Top8.50mm
- J4: footprint (none) -> Local_Connector_SocketHeader:SockHead_02x02_Pitch2.54mm_Bot3.10mm_Top8.50mm
- J5: footprint (none) -> Local_Connector_PinHeader:PinHead_01x03_Pitch2.54mm_Bot3.00mm_Top6.00mm_Shroud2.50mm
- P1, P2: footprint (none) -> Local_Module_Adafruit:Adafruit_BMP388
- P3, P4: footprint (none) -> Local_Module_Adafruit:Adafruit_BNO055
- Q1, Q2: footprint (none) -> Local_Package_SOT:SOT-23-3
- R1, R10, R11, R2, R3, R4, R5, R6, R7, R8, R9: footprint (none) -> Local_Resistor_SMD:Res_Film_0603
- TP1, TP2, TP3, TP4, TP5: footprint (none) -> Local_TestPoint:TestPoint_CircPad2.00mm_CircMsk2.50mm
- U1: footprint (none) -> Local_Package_SOIC:SOIC_28_Dim5.50x10.50x2.00mm_Pitch0.65mm
- U2: footprint (none) -> Local_Package_QFP:TQFP_08x08_Dim7.00x7.00x1.20mm_Pitch0.80mm
- Y1: footprint (none) -> Local_Crystal_SMD:Crystal_HC49-US
