File: CARL-Air-Brake-Peripheral-Devices-Hardware.kicad_pcb (KiCad board)
At the start: 2 copper layers, 65 x 56 mm, 53 parts, among them J1 ICSP, J2 USB, J3 Raspberry Pi, J4 Servo power, J5 Servo port, P1 BMP388, P2 BMP388, P3 BNO055, P4 BNO055, Q1 BSS138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

Commit message: Routed circuit board
Completed circuit design by routing all connections, and performed DRC.
Routing:
- net /SCL_3.3V: track 0.00 -> 85.4 mm, vias 0 -> 3
- net /SDA_3.3V: track 0.00 -> 82.4 mm, vias 0 -> 3
- net +6V: track 0.00 -> 72.3 mm, vias 0 -> 5
- net +3.3V: track 0.00 -> 54.8 mm, vias 0 -> 2
- net +5V: track 0.00 -> 42.7 mm, vias 0 -> 5
- net /SDA_5V: track 0.00 -> 41.3 mm, vias 0 -> 2
- net GND: track 0.00 -> 38.8 mm, vias 0 -> 12
- net /SCL_5V: track 0.00 -> 38.6 mm, vias 0 -> 2
- net Net-(D5-K): track 0.00 -> 32.2 mm, vias 0 -> 1
- net Net-(D4-K): track 0.00 -> 31.8 mm, vias 0 -> 1
- net /ICSP_MISO: track 0.00 -> 31.1 mm, vias 0 -> 1
- net /ICSP_RESET: track 0.00 -> 30.7 mm, vias 0 -> 3
- net VMCU: track 0.00 -> 23.6 mm, vias 0 -> 2
- net /ICSP_MOSI: track 0.00 -> 23.4 mm, vias 0 -> 1
- net /ICSP_SCK: track 0.00 -> 21.8 mm, vias 0 -> 1
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Other:
- board text added: "PWM"
